Commit message: fixed rotation axis

File: src/nexus_4wd_mecanum_description/urdf/nexus_4wd_mecanum.xacro (robot description, xacro)
@@ -188,5 +188,5 @@
       <origin xyz="0 0 0" rpy="0 0 0" />
       <geometry>
-        <mesh filename="file://$(find nexus_4wd_mecanum_description)/meshes/mecanum_wheel_right.STL" scale="0.001 0.001 0.001"/>
+        <mesh filename="file://$(find nexus_4wd_mecanum_description)/meshes/mecanum_wheel_left.STL" scale="0.001 0.001 0.001"/>
       </geometry>
       <material name="light_grey" />
@@ -211,5 +211,5 @@
     <parent link="upper_right_wheel_shaft"/>
     <child link="upper_right_wheel" />
-    <axis xyz="0 1 0"/>
+    <axis xyz="0 -1 0"/>
   </joint>
   <link name="upper_right_wheel">
@@ -240,5 +240,5 @@
     <parent link="lower_right_wheel_shaft"/>
     <child link="lower_right_wheel" />
-    <axis xyz="0 1 0"/>
+    <axis xyz="0 -1 0"/>
   </joint>
   <link name="lower_right_wheel">
@@ -246,5 +246,5 @@
       <origin xyz="0 0 0" rpy="0 0 0" />
       <geometry>
-        <mesh filename="file://$(find nexus_4wd_mecanum_description)/meshes/mecanum_wheel_left.STL" scale="0.001 0.001 0.001"/>
+        <mesh filename="file://$(find nexus_4wd_mecanum_description)/meshes/mecanum_wheel_right.STL" scale="0.001 0.001 0.001"/>
       </geometry>
       <material name="light_grey" />
@@ -269,5 +269,4 @@
       <plugin>gazebo_ros2_control/GazeboSystem</plugin>
     </hardware>
-    <!-- Front Left Wheel -->
     <joint name="upper_left_wheel_joint">
       <command_interface name="velocity">
@@ -278,5 +277,4 @@
       <state_interface name="velocity"/>
     </joint>
-    <!-- Rear Left Wheel -->
     <joint name="lower_left_wheel_joint">
       <command_interface name="velocity">
@@ -287,5 +285,4 @@
       <state_interface name="velocity"/>
     </joint>
-    <!-- Front Right Wheel -->
     <joint name="upper_right_wheel_joint">
       <command_interface name="velocity">
@@ -296,5 +293,4 @@
       <state_interface name="velocity"/>
     </joint>
-    <!-- Rear Right Wheel -->
     <joint name="lower_right_wheel_joint">
       <command_interface name="velocity">
@@ -306,9 +302,7 @@
     </joint>
   </ros2_control>
-  <!-- Include sensor modules -->
   <xacro:include filename="imu.urdf.xacro"/>
   <xacro:include filename="realsense.urdf.xacro"/>
   <xacro:include filename="lidar.urdf.xacro"/>
-  <!-- Include Gazebo plugins -->
   <xacro:include filename="nexus_4wd_mecanum.gazebo"/>
   <xacro:include filename="imu.gazebo"/>
