Commit message: things are connected but need refinment

File: mecanum_in_gazebo/urdf/mec_rob.ros2_control.xacro (robot description, xacro)
@@ -38,4 +38,13 @@
         <param name="min">-50</param>
         <param name="max">50</param>
+      </command_interface>
+      <state_interface name="position"/>
+      <state_interface name="velocity"/>
+    </joint>
+        <!-- LIFT JOINT -->
+    <joint name="lift_joint">
+      <command_interface name="position">
+        <param name="min">0.0</param>
+        <param name="max">0.35</param>
       </command_interface>
       <state_interface name="position"/>

File: mecanum_in_gazebo/urdf/mec_rob.xacro (robot description, xacro)
@@ -11,4 +11,7 @@
 <xacro:include filename="imu.gazebo" />
 <xacro:include filename="imu.urdf.xacro" />
+<xacro:include filename="lift.xacro" />
+<xacro:include filename="lift_camera.xacro" />
+<xacro:include filename="lift_camera.gazebo" />
 <link name="base_link">
   <inertial>
@@ -31,4 +34,12 @@
   </collision>
 </link>
+<!-- Lift Assembly -->
+<xacro:lift parent="base_link" name="lift" origin_xyz="0 0 0.05" origin_rpy="0 0 0"/>
+<!-- Camera on Lift -->
+<xacro:lift_camera_sensor parent="lift_platform_link" name="lift_camera">
+  <origin xyz="0 0 0.10" rpy="0 0 0"/>
+</xacro:lift_camera_sensor>
+<!-- Gazebo Camera Plugin -->
+<xacro:lift_camera_gazebo name="lift_camera"/>
 <link name="wheel_frame_FL_1">
   <inertial>
@@ -1083,3 +1094,12 @@
 </xacro:imu_sensor>
 <xacro:imu_gazebo name="imu"/>
+<xacro:lift
+    parent="base_link"
+    name="lift"
+    origin_xyz="0 0 0.05"
+    origin_rpy="0 0 0"/>
+<xacro:lift_camera_sensor parent="lift_platform_link" name="lift_camera">
+  <origin xyz="0 0 0.10" rpy="0 0 0"/>
+</xacro:lift_camera_sensor>
+<xacro:lift_camera_gazebo name="lift_camera"/>
 </robot>
