Commit message: everything's working

File: mecanum_in_gazebo/urdf/lift.xacro (robot description, xacro)
@@ -30,5 +30,5 @@
       <origin xyz="${origin_xyz}" rpy="${origin_rpy}"/>
       <axis xyz="0 0 1"/>
-      <limit lower="0.0" upper="0.35" velocity="0.2" effort="200"/>
+      <limit lower="0.0" upper="3.0" velocity="0.2" effort="200"/>
     </joint>
   </xacro:macro>

File: mecanum_in_gazebo/urdf/mec_rob.xacro (robot description, xacro)
@@ -34,12 +34,4 @@
   </collision>
 </link>
-<!-- Lift Assembly -->
-<xacro:lift parent="base_link" name="lift" origin_xyz="0 0 0.05" origin_rpy="0 0 0"/>
-<!-- Camera on Lift -->
-<xacro:lift_camera_sensor parent="lift_platform_link" name="lift_camera">
-  <origin xyz="0 0 0.10" rpy="0 0 0"/>
-</xacro:lift_camera_sensor>
-<!-- Gazebo Camera Plugin -->
-<xacro:lift_camera_gazebo name="lift_camera"/>
 <link name="wheel_frame_FL_1">
   <inertial>
