Commit message: tuned nav params

File: src/mecanum_in_gazebo/urdf/mec_rob.xacro (robot description, xacro)
@@ -1078,5 +1078,5 @@
 </joint>
 <xacro:lidar_sensor parent="base_link" name="lidar">
-  <origin xyz="0 0 0.08" rpy="0 0 0"/>
+  <origin xyz="0.35 0 0.08" rpy="0 0 0"/>
 </xacro:lidar_sensor>
 <xacro:lidar_gazebo name="lidar"/>
