Commit message: everything works

File: src/mecanum_in_gazebo/urdf/lift_camera.xacro (robot description, xacro)
@@ -30,5 +30,5 @@
         <parent link="lift_platform_link"/>
         <child link="lift_camera_link"/>
-        <origin xyz="0 0 0.07" rpy="0 0 0"/>
+        <origin xyz="0 0 0.07" rpy="0 0 1.57"/>
     </joint>
   </xacro:macro>
