Commit message: updates, lift joint added

File: warehouse/mecanum_in_gazebo/urdf/mec_rob.ros2_control.xacro (robot description, xacro)
@@ -42,5 +42,5 @@
       <state_interface name="velocity"/>
     </joint>
-           <!-- LIFT JOINT -->
+        <!-- LIFT JOINT -->
     <joint name="lift_joint">
       <command_interface name="position">
@@ -56,5 +56,38 @@
     <plugin filename="libgazebo_ros2_control.so" name="gazebo_ros2_control">
       <parameters>$(arg controller_config_file)</parameters>
+      <ros>
+        <namespace>/</namespace>
+        <remapping>/clock:=/clock</remapping>
+      </ros>
     </plugin>
+    <plugin name="p3d_base_controller" filename="libgazebo_ros_p3d.so">
+    <ros>
+      <namespace>/</namespace>
+      <remapping>odom:=odom</remapping>
+      <remapping>/clock:=/clock</remapping>
+    </ros>
+    <update_rate>50.0</update_rate>
+    <body_name>base_link</body_name>
+    <frame_name>odom</frame_name>
+    <xyz_offset>0 0 0</xyz_offset>
+    <rpy_offset>0 0 0</rpy_offset>
+    <gaussian_noise>0.01</gaussian_noise>
+  </plugin>
+    <!-- <plugin name="gazebo_ros_planar_move" filename="libgazebo_ros_planar_move.so">
+      <ros>
+        <namespace>/</namespace>
+        <remapping>cmd_vel:=cmd_vel</remapping>
+        <remapping>odom:=odom</remapping>
+      </ros>
+      <update_rate>50</update_rate>
+      <publish_rate>50</publish_rate>
+      <publish_odom>true</publish_odom>
+      <publish_odom_tf>true</publish_odom_tf>
+      <odometry_frame>odom</odometry_frame>
+      <robot_base_frame>base_link</robot_base_frame>
+      <covariance_x>0.0001</covariance_x>
+      <covariance_y>0.0001</covariance_y>
+      <covariance_yaw>0.01</covariance_yaw>
+    </plugin> -->
   </gazebo>
 </robot>

File: warehouse/mecanum_in_gazebo/urdf/mec_rob.xacro (robot description, xacro)
@@ -1,12 +1,5 @@
 <?xml version="1.0" ?>
 <robot name="mec_rob" xmlns:xacro="http://www.ros.org/wiki/xacro">
-<!-- <xacro:include filename="$(find mecanum_description)/urdf/mec_rob.ros2_control.xacro"/> -->
-<xacro:arg name="use_sim" default="true"/>
-<xacro:if value="$(arg use_sim)">
-  <xacro:include filename="$(find mecanum_description)/urdf/mec_rob.ros2_control.xacro"/>
-</xacro:if>
-<xacro:unless value="$(arg use_sim)">
-  <xacro:include filename="$(find mecanum_description)/urdf/mec_rob.ros2_control.hardware.xacro"/>
-</xacro:unless>
+<xacro:include filename="$(find mecanum_in_gazebo)/urdf/mec_rob.ros2_control.xacro"/>
 <xacro:include filename="lidar.xacro" />
 <xacro:include filename="lidar.gazebo" />
@@ -17,5 +10,5 @@
 <xacro:include filename="mec_rob.gazebo" />
 <xacro:include filename="imu.gazebo" />
-<xacro:include filename="imu.xacro" />
+<xacro:include filename="imu.urdf.xacro" />
 <xacro:include filename="lift.xacro" />
 <xacro:include filename="lift_camera.xacro" />
@@ -30,5 +23,5 @@
     <origin xyz="0 0 0" rpy="0 0 0"/>
     <geometry>
-      <mesh filename="file://$(find mecanum_description)/meshes/base_link.stl" scale="0.001 0.001 0.001"/>
+      <mesh filename="file://$(find mecanum_in_gazebo)/meshes/base_link.stl" scale="0.001 0.001 0.001"/>
     </geometry>
     <material name="silver"/>
@@ -37,5 +30,5 @@
     <origin xyz="0 0 0" rpy="0 0 0"/>
     <geometry>
-      <mesh filename="file://$(find mecanum_description)/meshes/base_link.stl" scale="0.001 0.001 0.001"/>
+      <mesh filename="file://$(find mecanum_in_gazebo)/meshes/base_link.stl" scale="0.001 0.001 0.001"/>
     </geometry>
   </collision>
@@ -50,5 +43,5 @@
     <origin xyz="-0.125 -0.15 -0.0" rpy="0 0 0"/>
     <geometry>
-      <mesh filename="file://$(find mecanum_description)/meshes/wheel_frame_FL_1.stl" scale="0.001 0.001 0.001"/>
+      <mesh filename="file://$(find mecanum_in_gazebo)/meshes/wheel_frame_FL_1.stl" scale="0.001 0.001 0.001"/>
     </geometry>
     <material name="silver"/>
@@ -57,5 +50,5 @@
     <origin xyz="-0.125 -0.15 -0.0" rpy="0 0 0"/>
     <geometry>
-      <mesh filename="file://$(find mecanum_description)/meshes/wheel_frame_FL_1.stl" scale="0.001 0.001 0.001"/>
+      <mesh filename="file://$(find mecanum_in_gazebo)/meshes/wheel_frame_FL_1.stl" scale="0.001 0.001 0.001"/>
     </geometry>
   </collision>
@@ -70,5 +63,5 @@
     <origin xyz="-0.142316 -0.142881 -0.04" rpy="0 0 0"/>
     <geometry>
-      <mesh filename="file://$(find mecanum_description)/meshes/roller_14_1.stl" scale="0.001 0.001 0.001"/>
+      <mesh filename="file://$(find mecanum_in_gazebo)/meshes/roller_14_1.stl" scale="0.001 0.001 0.001"/>
     </geometry>
     <material name="silver"/>
@@ -77,5 +70,5 @@
     <origin xyz="-0.142316 -0.142881 -0.04" rpy="0 0 0"/>
     <geometry>
-      <mesh filename="file://$(find mecanum_description)/meshes/roller_14_1.stl" scale="0.001 0.001 0.001"/>
+      <mesh filename="file://$(find mecanum_in_gazebo)/meshes/roller_14_1.stl" scale="0.001 0.001 0.001"/>
     </geometry>
   </collision>
@@ -90,5 +83,5 @@
     <origin xyz="-0.163976 -0.142881 -0.019512" rpy="0 0 0"/>
     <geometry>
-      <mesh filename="file://$(find mecanum_description)/meshes/roller_16_1.stl" scale="0.001 0.001 0.001"/>
+      <mesh filename="file://$(find mecanum_in_gazebo)/meshes/roller_16_1.stl" scale="0.001 0.001 0.001"/>
     </geometry>
     <material name="silver"/>
@@ -97,5 +90,5 @@
     <origin xyz="-0.163976 -0.142881 -0.019512" rpy="0 0 0"/>
     <geometry>
-      <mesh filename="file://$(find mecanum_description)/meshes/roller_16_1.stl" scale="0.001 0.001 0.001"/>
+      <mesh filename="file://$(find mecanum_in_gazebo)/meshes/roller_16_1.stl" scale="0.001 0.001 0.001"/>
     </geometry>
   </collision>
@@ -110,5 +103,5 @@
     <origin xyz="-0.167394 -0.142914 0.010075" rpy="0 0 0"/>
     <geometry>
-      <mesh filename="file://$(find mecanum_description)/meshes/roller_13_1.stl" scale="0.001 0.001 0.001"/>
+      <mesh filename="file://$(find mecanum_in_gazebo)/meshes/roller_13_1.stl" scale="0.001 0.001 0.001"/>
     </geometry>
     <material name="silver"/>
@@ -117,5 +110,5 @@
     <origin xyz="-0.167394 -0.142914 0.010075" rpy="0 0 0"/>
     <geometry>
-      <mesh filename="file://$(find mecanum_description)/meshes/roller_13_1.stl" scale="0.001 0.001 0.001"/>
+      <mesh filename="file://$(find mecanum_in_gazebo)/meshes/roller_13_1.stl" scale="0.001 0.001 0.001"/>
     </geometry>
   </collision>
@@ -130,5 +123,5 @@
     <origin xyz="-0.150999 -0.142914 0.034968" rpy="0 0 0"/>
     <geometry>
-      <mesh filename="file://$(find mecanum_description)/meshes/roller_12_1.stl" scale="0.001 0.001 0.001"/>
+      <mesh filename="file://$(find mecanum_in_gazebo)/meshes/roller_12_1.stl" scale="0.001 0.001 0.001"/>
     </geometry>
     <material name="silver"/>
@@ -137,5 +130,5 @@
     <origin xyz="-0.150999 -0.142914 0.034968" rpy="0 0 0"/>
     <geometry>
-      <mesh filename="file://$(find mecanum_description)/meshes/roller_12_1.stl" scale="0.001 0.001 0.001"/>
+      <mesh filename="file://$(find mecanum_in_gazebo)/meshes/roller_12_1.stl" scale="0.001 0.001 0.001"/>
     </geometry>
   </collision>
@@ -150,5 +143,5 @@
     <origin xyz="-0.12244 -0.142914 0.043499" rpy="0 0 0"/>
     <geometry>
-      <mesh filename="file://$(find mecanum_description)/meshes/roller_15_1.stl" scale="0.001 0.001 0.001"/>
+      <mesh filename="file://$(find mecanum_in_gazebo)/meshes/roller_15_1.stl" scale="0.001 0.001 0.001"/>
     </geometry>
     <material name="silver"/>
@@ -157,5 +150,5 @@
     <origin xyz="-0.12244 -0.142914 0.043499" rpy="0 0 0"/>
     <geometry>
-      <mesh filename="file://$(find mecanum_description)/meshes/roller_15_1.stl" scale="0.001 0.001 0.001"/>
+      <mesh filename="file://$(find mecanum_in_gazebo)/meshes/roller_15_1.stl" scale="0.001 0.001 0.001"/>
     </geometry>
   </collision>
@@ -170,5 +163,5 @@
     <origin xyz="-0.095078 -0.142914 0.031676" rpy="0 0 0"/>
     <geometry>
-      <mesh filename="file://$(find mecanum_description)/meshes/roller_17_1.stl" scale="0.001 0.001 0.001"/>
+      <mesh filename="file://$(find mecanum_in_gazebo)/meshes/roller_17_1.stl" scale="0.001 0.001 0.001"/>
     </geometry>
     <material name="silver"/>
@@ -177,5 +170,5 @@
     <origin xyz="-0.095078 -0.142914 0.031676" rpy="0 0 0"/>
     <geometry>
-      <mesh filename="file://$(find mecanum_description)/meshes/roller_17_1.stl" scale="0.001 0.001 0.001"/>
+      <mesh filename="file://$(find mecanum_in_gazebo)/meshes/roller_17_1.stl" scale="0.001 0.001 0.001"/>
     </geometry>
   </collision>
@@ -190,5 +183,5 @@
     <origin xyz="-0.081717 -0.142914 0.005032" rpy="0 0 0"/>
     <geometry>
-      <mesh filename="file://$(find mecanum_description)/meshes/roller_18_1.stl" scale="0.001 0.001 0.001"/>
+      <mesh filename="file://$(find mecanum_in_gazebo)/meshes/roller_18_1.stl" scale="0.001 0.001 0.001"/>
     </geometry>
     <material name="silver"/>
@@ -197,5 +190,5 @@
     <origin xyz="-0.081717 -0.142914 0.005032" rpy="0 0 0"/>
     <geometry>
-      <mesh filename="file://$(find mecanum_description)/meshes/roller_18_1.stl" scale="0.001 0.001 0.001"/>
+      <mesh filename="file://$(find mecanum_in_gazebo)/meshes/roller_18_1.stl" scale="0.001 0.001 0.001"/>
     </geometry>
   </collision>
@@ -210,5 +203,5 @@
     <origin xyz="-0.088609 -0.142914 -0.023967" rpy="0 0 0"/>
     <geometry>
-      <mesh filename="file://$(find mecanum_description)/meshes/roller_10_1.stl" scale="0.001 0.001 0.001"/>
+      <mesh filename="file://$(find mecanum_in_gazebo)/meshes/roller_10_1.stl" scale="0.001 0.001 0.001"/>
     </geometry>
     <material name="silver"/>
@@ -217,5 +210,5 @@
     <origin xyz="-0.088609 -0.142914 -0.023967" rpy="0 0 0"/>
     <geometry>
-      <mesh filename="file://$(find mecanum_description)/meshes/roller_10_1.stl" scale="0.001 0.001 0.001"/>
+      <mesh filename="file://$(find mecanum_in_gazebo)/meshes/roller_10_1.stl" scale="0.001 0.001 0.001"/>
     </geometry>
   </collision>
@@ -230,5 +223,5 @@
     <origin xyz="-0.112528 -0.142914 -0.041751" rpy="0 0 0"/>
     <geometry>
-      <mesh filename="file://$(find mecanum_description)/meshes/roller_11_1.stl" scale="0.001 0.001 0.001"/>
+      <mesh filename="file://$(find mecanum_in_gazebo)/meshes/roller_11_1.stl" scale="0.001 0.001 0.001"/>
     </geometry>
     <material name="silver"/>
@@ -237,5 +230,5 @@
     <origin xyz="-0.112528 -0.142914 -0.041751" rpy="0 0 0"/>
     <geometry>
-      <mesh filename="file://$(find mecanum_description)/meshes/roller_11_1.stl" scale="0.001 0.001 0.001"/>
+      <mesh filename="file://$(find mecanum_in_gazebo)/meshes/roller_11_1.stl" scale="0.001 0.001 0.001"/>
     </geometry>
   </collision>
@@ -250,5 +243,5 @@
     <origin xyz="-0.125 0.15 -0.0" rpy="0 0 0"/>
     <geometry>
-      <mesh filename="file://$(find mecanum_description)/meshes/wheel_frame_FR_1.stl" scale="0.001 0.001 0.001"/>
+      <mesh filename="file://$(find mecanum_in_gazebo)/meshes/wheel_frame_FR_1.stl" scale="0.001 0.001 0.001"/>
     </geometry>
     <material name="silver"/>
@@ -257,5 +250,5 @@
     <origin xyz="-0.125 0.15 -0.0" rpy="0 0 0"/>
     <geometry>
-      <mesh filename="file://$(find mecanum_description)/meshes/wheel_frame_FR_1.stl" scale="0.001 0.001 0.001"/>
+      <mesh filename="file://$(find mecanum_in_gazebo)/meshes/wheel_frame_FR_1.stl" scale="0.001 0.001 0.001"/>
     </geometry>
   </collision>
@@ -270,5 +263,5 @@
     <origin xyz="-0.107684 0.109619 -0.04" rpy="0 0 0"/>
     <geometry>
-      <mesh filename="file://$(find mecanum_description)/meshes/roller_7_1.stl" scale="0.001 0.001 0.001"/>
+      <mesh filename="file://$(find mecanum_in_gazebo)/meshes/roller_7_1.stl" scale="0.001 0.001 0.001"/>
     </geometry>
     <material name="silver"/>
@@ -277,5 +270,5 @@
     <origin xyz="-0.107684 0.109619 -0.04" rpy="0 0 0"/>
     <geometry>
-      <mesh filename="file://$(find mecanum_description)/meshes/roller_7_1.stl" scale="0.001 0.001 0.001"/>
+      <mesh filename="file://$(find mecanum_in_gazebo)/meshes/roller_7_1.stl" scale="0.001 0.001 0.001"/>
     </geometry>
   </collision>
@@ -290,5 +283,5 @@
     <origin xyz="-0.137447 0.109619 -0.041772" rpy="0 0 0"/>
     <geometry>
-      <mesh filename="file://$(find mecanum_description)/meshes/roller_5_1.stl" scale="0.001 0.001 0.001"/>
+      <mesh filename="file://$(find mecanum_in_gazebo)/meshes/roller_5_1.stl" scale="0.001 0.001 0.001"/>
     </geometry>
     <material name="silver"/>
@@ -297,5 +290,5 @@
     <origin xyz="-0.137447 0.109619 -0.041772" rpy="0 0 0"/>
     <geometry>
-      <mesh filename="file://$(find mecanum_description)/meshes/roller_5_1.stl" scale="0.001 0.001 0.001"/>
+      <mesh filename="file://$(find mecanum_in_gazebo)/meshes/roller_5_1.stl" scale="0.001 0.001 0.001"/>
     </geometry>
   </collision>
@@ -310,5 +303,5 @@
     <origin xyz="-0.161385 0.109619 -0.023998" rpy="0 0 0"/>
     <geometry>
-      <mesh filename="file://$(find mecanum_description)/meshes/roller_3_1.stl" scale="0.001 0.001 0.001"/>
+      <mesh filename="file://$(find mecanum_in_gazebo)/meshes/roller_3_1.stl" scale="0.001 0.001 0.001"/>
     </geometry>
     <material name="silver"/>
@@ -317,5 +310,5 @@
     <origin xyz="-0.161385 0.109619 -0.023998" rpy="0 0 0"/>
     <geometry>
-      <mesh filename="file://$(find mecanum_description)/meshes/roller_3_1.stl" scale="0.001 0.001 0.001"/>
+      <mesh filename="file://$(find mecanum_in_gazebo)/meshes/roller_3_1.stl" scale="0.001 0.001 0.001"/>
     </geometry>
   </collision>
@@ -330,5 +323,5 @@
     <origin xyz="-0.168299 0.109619 0.005004" rpy="0 0 0"/>
     <geometry>
-      <mesh filename="file://$(find mecanum_description)/meshes/roller_6_1.stl" scale="0.001 0.001 0.001"/>
+      <mesh filename="file://$(find mecanum_in_gazebo)/meshes/roller_6_1.stl" scale="0.001 0.001 0.001"/>
     </geometry>
     <material name="silver"/>
@@ -337,5 +330,5 @@
     <origin xyz="-0.168299 0.109619 0.005004" rpy="0 0 0"/>
     <geometry>
-      <mesh filename="file://$(find mecanum_description)/meshes/roller_6_1.stl" scale="0.001 0.001 0.001"/>
+      <mesh filename="file://$(find mecanum_in_gazebo)/meshes/roller_6_1.stl" scale="0.001 0.001 0.001"/>
     </geometry>
   </collision>
@@ -350,5 +343,5 @@
     <origin xyz="-0.154952 0.109619 0.031665" rpy="0 0 0"/>
     <geometry>
-      <mesh filename="file://$(find mecanum_description)/meshes/roller_8_1.stl" scale="0.001 0.001 0.001"/>
+      <mesh filename="file://$(find mecanum_in_gazebo)/meshes/roller_8_1.stl" scale="0.001 0.001 0.001"/>
     </geometry>
     <material name="silver"/>
@@ -357,5 +350,5 @@
     <origin xyz="-0.154952 0.109619 0.031665" rpy="0 0 0"/>
     <geometry>
-      <mesh filename="file://$(find mecanum_description)/meshes/roller_8_1.stl" scale="0.001 0.001 0.001"/>
+      <mesh filename="file://$(find mecanum_in_gazebo)/meshes/roller_8_1.stl" scale="0.001 0.001 0.001"/>
     </geometry>
   </collision>
@@ -370,5 +363,5 @@
     <origin xyz="-0.127591 0.109619 0.04351" rpy="0 0 0"/>
     <geometry>
-      <mesh filename="file://$(find mecanum_description)/meshes/roller_9_1.stl" scale="0.001 0.001 0.001"/>
+      <mesh filename="file://$(find mecanum_in_gazebo)/meshes/roller_9_1.stl" scale="0.001 0.001 0.001"/>
     </geometry>
     <material name="silver"/>
@@ -377,5 +370,5 @@
     <origin xyz="-0.127591 0.109619 0.04351" rpy="0 0 0"/>
     <geometry>
-      <mesh filename="file://$(find mecanum_description)/meshes/roller_9_1.stl" scale="0.001 0.001 0.001"/>
+      <mesh filename="file://$(find mecanum_in_gazebo)/meshes/roller_9_1.stl" scale="0.001 0.001 0.001"/>
     </geometry>
   </collision>
@@ -390,5 +383,5 @@
     <origin xyz="-0.099017 0.109619 0.034996" rpy="0 0 0"/>
     <geometry>
-      <mesh filename="file://$(find mecanum_description)/meshes/roller_4_1.stl" scale="0.001 0.001 0.001"/>
+      <mesh filename="file://$(find mecanum_in_gazebo)/meshes/roller_4_1.stl" scale="0.001 0.001 0.001"/>
     </geometry>
     <material name="silver"/>
@@ -397,5 +390,5 @@
     <origin xyz="-0.099017 0.109619 0.034996" rpy="0 0 0"/>
     <geometry>
-      <mesh filename="file://$(find mecanum_description)/meshes/roller_4_1.stl" scale="0.001 0.001 0.001"/>
+      <mesh filename="file://$(find mecanum_in_gazebo)/meshes/roller_4_1.stl" scale="0.001 0.001 0.001"/>
     </geometry>
   </collision>
@@ -410,5 +403,5 @@
     <origin xyz="-0.082601 0.109619 0.010107" rpy="0 0 0"/>
     <geometry>
-      <mesh filename="file://$(find mecanum_description)/meshes/roller_1_1.stl" scale="0.001 0.001 0.001"/>
+      <mesh filename="file://$(find mecanum_in_gazebo)/meshes/roller_1_1.stl" scale="0.001 0.001 0.001"/>
     </geometry>
     <material name="silver"/>
@@ -417,5 +410,5 @@
     <origin xyz="-0.082601 0.109619 0.010107" rpy="0 0 0"/>
     <geometry>
-      <mesh filename="file://$(find mecanum_description)/meshes/roller_1_1.stl" scale="0.001 0.001 0.001"/>
+      <mesh filename="file://$(find mecanum_in_gazebo)/meshes/roller_1_1.stl" scale="0.001 0.001 0.001"/>
     </geometry>
   </collision>
@@ -430,5 +423,5 @@
     <origin xyz="-0.086024 0.109619 -0.019512" rpy="0 0 0"/>
     <geometry>
-      <mesh filename="file://$(find mecanum_description)/meshes/roller_2_1.stl" scale="0.001 0.001 0.001"/>
+      <mesh filename="file://$(find mecanum_in_gazebo)/meshes/roller_2_1.stl" scale="0.001 0.001 0.001"/>
     </geometry>
     <material name="silver"/>
@@ -437,5 +430,5 @@
     <origin xyz="-0.086024 0.109619 -0.019512" rpy="0 0 0"/>
     <geometry>
-      <mesh filename="file://$(find mecanum_description)/meshes/roller_2_1.stl" scale="0.001 0.001 0.001"/>
+      <mesh filename="file://$(find mecanum_in_gazebo)/meshes/roller_2_1.stl" scale="0.001 0.001 0.001"/>
     </geometry>
   </collision>
@@ -450,5 +443,5 @@
     <origin xyz="0.125 -0.15 -0.0" rpy="0 0 0"/>
     <geometry>
-      <mesh filename="file://$(find mecanum_description)/meshes/wheel_frame_BL_1.stl" scale="0.001 0.001 0.001"/>
+      <mesh filename="file://$(find mecanum_in_gazebo)/meshes/wheel_frame_BL_1.stl" scale="0.001 0.001 0.001"/>
     </geometry>
     <material name="silver"/>
@@ -457,5 +450,5 @@
     <origin xyz="0.125 -0.15 -0.0" rpy="0 0 0"/>
     <geometry>
-      <mesh filename="file://$(find mecanum_description)/meshes/wheel_frame_BL_1.stl" scale="0.001 0.001 0.001"/>
+      <mesh filename="file://$(find mecanum_in_gazebo)/meshes/wheel_frame_BL_1.stl" scale="0.001 0.001 0.001"/>
     </geometry>
   </collision>
@@ -470,5 +463,5 @@
     <origin xyz="0.142316 -0.142881 -0.04" rpy="0 0 0"/>
     <geometry>
-      <mesh filename="file://$(find mecanum_description)/meshes/roller_23_1.stl" scale="0.001 0.001 0.001"/>
+      <mesh filename="file://$(find mecanum_in_gazebo)/meshes/roller_23_1.stl" scale="0.001 0.001 0.001"/>
     </geometry>
     <material name="silver"/>
@@ -477,5 +470,5 @@
     <origin xyz="0.142316 -0.142881 -0.04" rpy="0 0 0"/>
     <geometry>
-      <mesh filename="file://$(find mecanum_description)/meshes/roller_23_1.stl" scale="0.001 0.001 0.001"/>
+      <mesh filename="file://$(find mecanum_in_gazebo)/meshes/roller_23_1.stl" scale="0.001 0.001 0.001"/>
     </geometry>
   </collision>
@@ -490,5 +483,5 @@
     <origin xyz="0.112553 -0.142881 -0.041772" rpy="0 0 0"/>
     <geometry>
-      <mesh filename="file://$(find mecanum_description)/meshes/roller_22_1.stl" scale="0.001 0.001 0.001"/>
+      <mesh filename="file://$(find mecanum_in_gazebo)/meshes/roller_22_1.stl" scale="0.001 0.001 0.001"/>
     </geometry>
     <material name="silver"/>
@@ -497,5 +490,5 @@
     <origin xyz="0.112553 -0.142881 -0.041772" rpy="0 0 0"/>
     <geometry>
-      <mesh filename="file://$(find mecanum_description)/meshes/roller_22_1.stl" scale="0.001 0.001 0.001"/>
+      <mesh filename="file://$(find mecanum_in_gazebo)/meshes/roller_22_1.stl" scale="0.001 0.001 0.001"/>
     </geometry>
   </collision>
@@ -510,5 +503,5 @@
     <origin xyz="0.088615 -0.142881 -0.023998" rpy="0 0 0"/>
     <geometry>
-      <mesh filename="file://$(find mecanum_description)/meshes/roller_25_1.stl" scale="0.001 0.001 0.001"/>
+      <mesh filename="file://$(find mecanum_in_gazebo)/meshes/roller_25_1.stl" scale="0.001 0.001 0.001"/>
     </geometry>
     <material name="silver"/>
@@ -517,5 +510,5 @@
     <origin xyz="0.088615 -0.142881 -0.023998" rpy="0 0 0"/>
     <geometry>
-      <mesh filename="file://$(find mecanum_description)/meshes/roller_25_1.stl" scale="0.001 0.001 0.001"/>
+      <mesh filename="file://$(find mecanum_in_gazebo)/meshes/roller_25_1.stl" scale="0.001 0.001 0.001"/>
     </geometry>
   </collision>
@@ -530,5 +523,5 @@
     <origin xyz="0.081701 -0.142881 0.005004" rpy="0 0 0"/>
     <geometry>
-      <mesh filename="file://$(find mecanum_description)/meshes/roller_21_1.stl" scale="0.001 0.001 0.001"/>
+      <mesh filename="file://$(find mecanum_in_gazebo)/meshes/roller_21_1.stl" scale="0.001 0.001 0.001"/>
     </geometry>
     <material name="silver"/>
@@ -537,5 +530,5 @@
     <origin xyz="0.081701 -0.142881 0.005004" rpy="0 0 0"/>
     <geometry>
-      <mesh filename="file://$(find mecanum_description)/meshes/roller_21_1.stl" scale="0.001 0.001 0.001"/>
+      <mesh filename="file://$(find mecanum_in_gazebo)/meshes/roller_21_1.stl" scale="0.001 0.001 0.001"/>
     </geometry>
   </collision>
@@ -550,5 +543,5 @@
     <origin xyz="0.095048 -0.142881 0.031665" rpy="0 0 0"/>
     <geometry>
-      <mesh filename="file://$(find mecanum_description)/meshes/roller_26_1.stl" scale="0.001 0.001 0.001"/>
+      <mesh filename="file://$(find mecanum_in_gazebo)/meshes/roller_26_1.stl" scale="0.001 0.001 0.001"/>
     </geometry>
     <material name="silver"/>
@@ -557,5 +550,5 @@
     <origin xyz="0.095048 -0.142881 0.031665" rpy="0 0 0"/>
     <geometry>
-      <mesh filename="file://$(find mecanum_description)/meshes/roller_26_1.stl" scale="0.001 0.001 0.001"/>
+      <mesh filename="file://$(find mecanum_in_gazebo)/meshes/roller_26_1.stl" scale="0.001 0.001 0.001"/>
     </geometry>
   </collision>
@@ -570,5 +563,5 @@
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